File: ne5532_headphones_amp.sch (KiCad schematic (older format))
At the start: 30 parts, among them J1 AudioJack3_Ground, J2 AudioJack3_Ground, Q1 BD140, Q2 BD139, Q3 BD139, Q4 BD140, U1 NE5532

Commit message: board layout
Parts:
- removed J1, J2: AudioJack3_Ground, symbol Connector:AudioJack3_Ground
- added J1, J2: JACK_TRS_3PINS, lm386_headphones_amplifier:3.5mm_stereo_TRS_jack, symbol JACK_TRS:JACK_TRS_3PINS
- added J3: Conn_01x03_Male, Connector_PinHeader_2.54mm:PinHeader_1x03_P2.54mm_Vertical, symbol Connector:Conn_01x03_Male
- C1, C2: footprint (none) -> Capacitor_THT:CP_Radial_D5.0mm_P2.50mm
- C3, C4: footprint (none) -> Capacitor_THT:C_Disc_D3.0mm_W2.0mm_P2.50mm
- CP1: renamed from 10uF1; value CP1 -> 10u; footprint (none) -> Capacitor_THT:CP_Radial_D5.0mm_P2.00mm
- CP2: renamed from 10uF2; value CP1 -> 10u; footprint (none) -> Capacitor_THT:CP_Radial_D5.0mm_P2.00mm
- R1, R2: footprint (none) -> Resistor_THT:R_Axial_DIN0207_L6.3mm_D2.5mm_P10.16mm_Horizontal
- R10: renamed from 10R2; value R_Small -> 10R; footprint (none) -> Resistor_THT:R_Axial_DIN0207_L6.3mm_D2.5mm_P10.16mm_Horizontal
- R11: renamed from 10R3; value R_Small -> 10R; footprint (none) -> Resistor_THT:R_Axial_DIN0207_L6.3mm_D2.5mm_P10.16mm_Horizontal
- R12: renamed from 10R4; value R_Small -> 10R; footprint (none) -> Resistor_THT:R_Axial_DIN0207_L6.3mm_D2.5mm_P10.16mm_Horizontal
- R3: renamed from 1K1; value R -> 1K; footprint (none) -> Resistor_THT:R_Axial_DIN0207_L6.3mm_D2.5mm_P10.16mm_Horizontal
- R4: renamed from 1K2; value R -> 1K; footprint (none) -> Resistor_THT:R_Axial_DIN0207_L6.3mm_D2.5mm_P10.16mm_Horizontal
- R5: renamed from 4.7K1; value R -> 4.7K; footprint (none) -> Resistor_THT:R_Axial_DIN0207_L6.3mm_D2.5mm_P10.16mm_Horizontal
- R6: renamed from 4.7K2; value R -> 4.7K; footprint (none) -> Resistor_THT:R_Axial_DIN0207_L6.3mm_D2.5mm_P10.16mm_Horizontal
- R7: renamed from 4.7K3; value R -> 4.7K; footprint (none) -> Resistor_THT:R_Axial_DIN0207_L6.3mm_D2.5mm_P10.16mm_Horizontal
- R8: renamed from 4.7K4; value R -> 4.7K; footprint (none) -> Resistor_THT:R_Axial_DIN0207_L6.3mm_D2.5mm_P10.16mm_Horizontal
- R9: renamed from 10R1; value R_Small -> 10R; footprint (none) -> Resistor_THT:R_Axial_DIN0207_L6.3mm_D2.5mm_P10.16mm_Horizontal
- RV1: value R_POT_Dual -> 10K; footprint (none) -> Potentiometer_THT:Potentiometer_Alps_RK163_Dual_Horizontal
- U1: footprint (none) -> Package_DIP:DIP-8_W7.62mm_Socket
Connections:
- net +9V: now also J3.1 (Pin_1)
- net -9V: now also J3.3 (Pin_3)
- net GND: now also J1.1 (S), J2.1 (S), J3.2 (Pin_2)
- net JACK_R: now reaches RV1.6
- net JACK_R: now also J1.2 (R)
- net JACK_T: now reaches RV1.3
- net JACK_T: now also J1.3 (T)
- net JACK_OUT_R: now reaches R1.1, R10.1, R9.2
- net JACK_OUT_R: now also J2.2 (R)
- net JACK_OUT_T: now reaches R11.2, R12.1, R2.1
- net JACK_OUT_T: now also J2.3 (T)
